File: boards/6-led/wings-led-6.kicad_sch (KiCad schematic)
At the start: 0 parts

Commit message: boards: add 6-LED schematic (ERC-clean, netlist matches spec)
Authored wings-led-6.kicad_sch for a single 6-LED strip module:

- 6x SK9822-EC20 (APA102-2020 symbol, L1-L6) + 6x 100nF decoupling (C1-C6)
- 2x JST-GH 4-pin SMD (J1 IN, J2 OUT), wired per the canonical pinout
- +5V/GND rails, power symbols + PWR_FLAGs, net labels (SDI/CLK/D1-D5/CLK1-CLK5/SDO/CKO)
- footprints pre-assigned to the vendored wings-led-6 libraries
- wired by signal name per the APA102/SK9822 pin-number caveat

Validated with kicad-cli: sch erc = 0 violations; netlist matches boards/modules/6-led-schematic.md. Populated wings-led-6.kicad_pro (registers the root sheet).
Parts:
- added C1, C2, C3, C4, C5, C6: 100nF, wings-led-6:C_0603_1608Metric, symbol wings-led-6:C
- added J1: JST-GH 4p IN, wings-led-6:JST_GH_SM04B-GHS-TB_1x04-1MP_P1.25mm_Horizontal, symbol wings-led-6:Conn_01x04
- added J2: JST-GH 4p OUT, wings-led-6:JST_GH_SM04B-GHS-TB_1x04-1MP_P1.25mm_Horizontal, symbol wings-led-6:Conn_01x04
- added L1, L2, L3, L4, L5, L6: SK9822-EC20, wings-led-6:LED-APA102-2020, symbol wings-led-6:APA102-2020
Connections:
- new net +5V: C1.1, C2.1, C3.1, C4.1, C5.1, C6.1, J1.4 (Pin_4), J2.1 (Pin_1), L1.1 (VDD), L2.1 (VDD), L3.1 (VDD), L4.1 (VDD), L5.1 (VDD), L6.1 (VDD)
- new net CKO: J2.2 (Pin_2), L6.2 (CKO)
- new net CLK: J1.2 (Pin_2), L1.5 (CKI)
- new net CLK1: L1.2 (CKO), L2.5 (CKI)
- new net CLK2: L2.2 (CKO), L3.5 (CKI)
- new net CLK3: L3.2 (CKO), L4.5 (CKI)
- new net CLK4: L4.2 (CKO), L5.5 (CKI)
- new net CLK5: L5.2 (CKO), L6.5 (CKI)
- new net D1: L1.3 (SDO), L2.4 (SDI)
- new net D2: L2.3 (SDO), L3.4 (SDI)
- new net D3: L3.3 (SDO), L4.4 (SDI)
- new net D4: L4.3 (SDO), L5.4 (SDI)
- new net D5: L5.3 (SDO), L6.4 (SDI)
- new net GND: C1.2, C2.2, C3.2, C4.2, C5.2, C6.2, J1.1 (Pin_1), J2.4 (Pin_4), L1.6 (GND), L2.6 (GND), L3.6 (GND), L4.6 (GND), L5.6 (GND), L6.6 (GND)
- new net SDI: J1.3 (Pin_3), L1.4 (SDI)
- new net SDO: J2.3 (Pin_3), L6.3 (SDO)
Other:
- note added: "6-LED Strip Module - SK9822-EC20 x6"
- note added: "IN"
- note added: "OUT"

Commit message: updating kicad symbols
Parts:
- removed L1, L2, L3, L4, L5, L6: SK9822-EC20, wings-led-6:LED-APA102-2020, symbol wings-led-6:APA102-2020
- added L1, L2, L3, L4, L5, L6: SK9822-EC20, easyeda2kicad:LED-SMD_6P-L2.0-W2.0-P0.80-TL, symbol easyeda2kicad:SK9822-EC20
Connections:
- net CKO is gone; now on net +5V: J2.2 (Pin_2)
- net SDI is gone; now on net CLK: J1.3 (Pin_3)
- net +5V: now also L1.5 (VDD), L1.6 (CKO), L2.4 (CKL), L2.5 (VDD), L2.6 (CKO), L3.4 (CKL), L3.5 (VDD), L3.6 (CKO), L4.4 (CKL), L4.5 (VDD), L4.6 (CKO), L5.4 (CKL), L5.5 (VDD), L5.6 (CKO), L6.4 (CKL), L6.5 (VDD), L6.6 (CKO)
- net CLK: now also L1.4 (CKL); no longer J1.2 (Pin_2)
- net GND: now also J1.2 (Pin_2), L1.1 (SDO), L1.2 (GND), L1.3 (SDI), L2.1 (SDO), L2.2 (GND), L2.3 (SDI), L3.1 (SDO), L3.2 (GND), L3.3 (SDI), L4.1 (SDO), L4.2 (GND), L4.3 (SDI), L5.1 (SDO), L5.2 (GND), L5.3 (SDI), L6.2 (GND), L6.3 (SDI)
- net SDO: now also L6.1 (SDO)
