File: boards/2020-leds/SK9822-EC20-strip.kicad_sch (KiCad schematic)
At the start: 0 parts

Commit message: led strip: gen_schematic SKU set 7-12 + C1 bulk cap; project fp-lib-table (17 footprint libs) fixing footprint resolution; KiCad board/schematic updates from footprint remap
Parts:
- added C1: 22uF, C12891:C1206, symbol wings:CL31A226KAHNNNE
- added J1: DATA-IN, C145992:CONN-SMD_ZH1.5-4P_SMD, symbol wings:ZH1.5-4PSMD
- added J2: DATA-OUT, C145992:CONN-SMD_ZH1.5-4P_SMD, symbol wings:ZH1.5-4PSMD
- added J3: PWR-TAP, C47647:CONN-SMD_2P-P2.00_PH2.0-SPWB, symbol wings:PH2.0-2PWB
- added L1, L10, L11, L12, L2, L3, L4, L5, L6, L7, L8, L9: SK9822-EC20, C2909059:LED-SMD_6P-L2.0-W2.0-P0.80-TL, symbol wings:SK9822-EC20
Connections:
- new net +5V: C1.1, J1.4, J2.1, J3.1, L1.5 (VDD), L10.5 (VDD), L11.5 (VDD), L12.5 (VDD), L2.5 (VDD), L3.5 (VDD), L4.5 (VDD), L5.5 (VDD), L6.5 (VDD), L7.5 (VDD), L8.5 (VDD), L9.5 (VDD)
- new net C0: L1.6 (CKO), L2.4 (CKL)
- new net C1: L2.6 (CKO), L3.4 (CKL)
- new net C10: L11.6 (CKO), L12.4 (CKL)
- new net C2: L3.6 (CKO), L4.4 (CKL)
- new net C3: L4.6 (CKO), L5.4 (CKL)
- new net C4: L5.6 (CKO), L6.4 (CKL)
- new net C5: L6.6 (CKO), L7.4 (CKL)
- new net C6: L7.6 (CKO), L8.4 (CKL)
- new net C7: L8.6 (CKO), L9.4 (CKL)
- new net C8: L10.4 (CKL), L9.6 (CKO)
- new net C9: L10.6 (CKO), L11.4 (CKL)
- new net CI: J1.2, L1.4 (CKL)
- new net CO: J2.3, L12.6 (CKO)
- new net D0: L1.1 (SDO), L2.3 (SDI)
- new net D1: L2.1 (SDO), L3.3 (SDI)
- new net D10: L11.1 (SDO), L12.3 (SDI)
- new net D2: L3.1 (SDO), L4.3 (SDI)
- new net D3: L4.1 (SDO), L5.3 (SDI)
- new net D4: L5.1 (SDO), L6.3 (SDI)
- new net D5: L6.1 (SDO), L7.3 (SDI)
- new net D6: L7.1 (SDO), L8.3 (SDI)
- new net D7: L8.1 (SDO), L9.3 (SDI)
- new net D8: L10.3 (SDI), L9.1 (SDO)
- new net D9: L10.1 (SDO), L11.3 (SDI)
- new net DI: J1.3, L1.3 (SDI)
- new net DO: J2.2, L12.1 (SDO)
- new net GND: C1.2, J1.1, J2.4, J3.2, L1.2 (GND), L10.2 (GND), L11.2 (GND), L12.2 (GND), L2.2 (GND), L3.2 (GND), L4.2 (GND), L5.2 (GND), L6.2 (GND), L7.2 (GND), L8.2 (GND), L9.2 (GND)
